File: Hank2.brd (EAGLE design)
At the start: 22.8 x 51.1 mm, 44 parts

Commit message: Wired SSR circuits
Parts:
- added MOUT: (no value), con-ptr500:AK300/10
- added SV1: (no value), con-lstb:MA09-1
- X1: value (none) -> 22-23-2091; device con-ptr500:AK300/9 -> con-molex:22-23-2091
- moved X1 267.8 mm to (-13.1, -702.7)
Connections:
- net N$14 renamed OUT5
- net N$18 renamed OUT6
- net N$22 renamed OUT7
- net N$27 renamed OUT8
- net N$31 renamed OUT1
- net N$35 renamed OUT2
- net N$39 renamed OUT3
- net N$43 renamed OUT4
- new net L1-1: MOUT.1, U$19.1, U$20.1, U$21.1, U$22.1
- new net L1-2: MOUT.6, U$16.1, U$17.1, U$18.1, U$8.1
- new net MOUT1: MOUT.2, U$19.2
- new net MOUT2: MOUT.3, U$20.2
- new net MOUT3: MOUT.4, U$21.2
- new net MOUT4: MOUT.5, U$22.2
- new net MOUT5: MOUT.7, U$8.2
- new net MOUT6: MOUT.8, U$16.2
- new net MOUT7: MOUT.9, U$17.2
- new net MOUT8: MOUT.10, U$18.2
Changed lines of the file:
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@@
 <element name="LED4" library="led" package="LED3MM" value="" x="-3.560903125" y="-409.554503125"/>
 <element name="R15" library="rcl" package="0204/7" value="" x="-20.84100625" y="-409.554503125"/>
-<element name="X1" library="con-ptr500" package="AK300/9" value="" x="-0.828903125" y="-435.123640625">
-<attribute name="MF" value="" x="-0.828903125" y="-435.123640625" size="1.778" layer="27" display="off"/>
-<attribute name="OC_FARNELL" value="unknown" x="-0.828903125" y="-435.123640625" size="1.778" layer="27" display="off"/>
-<attribute name="MPN" value="" x="-0.828903125" y="-435.123640625" size="1.778" layer="27" display="off"/>
-<attribute name="OC_NEWARK" value="unknown" x="-0.828903125" y="-435.123640625" size="1.778" layer="27" display="off"/>
-</element>
 <element name="U$19" library="HankLibraries" package="SSR_FOOTPRINT" value="SSR" x="-20.891753125" y="-494.0180875"/>
 <element name="R16" library="rcl" package="0204/7" value="" x="-20.84100625" y="-470.94411875"/>
@@
 <element name="LED8" library="led" package="LED3MM" value="" x="-3.560903125" y="-644.447175"/>
 <element name="R23" library="rcl" package="0204/7" value="" x="-20.84100625" y="-644.447175"/>
+<element name="MOUT" library="con-ptr500" package="AK300/10" value="" x="1.65780625" y="-670.0163125">
+<attribute name="MF" value="" x="1.65780625" y="-670.0163125" size="1.778" layer="27" display="off"/>
+<attribute name="OC_FARNELL" value="unknown" x="1.65780625" y="-670.0163125" size="1.778" layer="27" display="off"/>
+<attribute name="MPN" value="" x="1.65780625" y="-670.0163125" size="1.778" layer="27" display="off"/>
+<attribute name="OC_NEWARK" value="unknown" x="1.65780625" y="-670.0163125" size="1.778" layer="27" display="off"/>
+</element>
+<element name="SV1" library="con-lstb" package="MA09-1" value="" x="-12.966421875" y="-687.5501625">
+<attribute name="MF" value="" x="-12.966421875" y="-687.5501625" size="1.778" layer="27" display="off"/>
+<attribute name="OC_FARNELL" value="unknown" x="-12.966421875" y="-687.5501625" size="1.778" layer="27" display="off"/>
+<attribute name="MPN" value="" x="-12.966421875" y="-687.5501625" size="1.778" layer="27" display="off"/>
+<attribute name="OC_NEWARK" value="unknown" x="-12.966421875" y="-687.5501625" size="1.778" layer="27" display="off"/>
+</element>
+<element name="X1" library="con-molex" package="22-23-2091" value="22-23-2091" x="-13.09329375" y="-702.673421875">
+<attribute name="MF" value="MOLEX" x="-13.09329375" y="-702.673421875" size="1.778" layer="27" display="off"/>
+<attribute name="OC_FARNELL" value="1756827" x="-13.09329375" y="-702.673421875" size="1.778" layer="27" display="off"/>
+<attribute name="MPN" value="22-23-2091" x="-13.09329375" y="-702.673421875" size="1.778" layer="27" display="off"/>
+<attribute name="OC_NEWARK" value="56H0450" x="-13.09329375" y="-702.673421875" size="1.778" layer="27" display="off"/>
+</element>
 </elements>
 <signals>
@@
 <wire x1="-24.701753125" y1="-67.225775" x2="-17.03100625" y2="-233.420946875" width="0" layer="19" extent="1-1"/>
 </signal>
-<signal name="N$14">
+<signal name="OUT5">
 <contactref element="OK1" pad="1"/>
 </signal>
@@
 <wire x1="-17.03100625" y1="-409.554503125" x2="-6.876084375" y2="-201.41046875" width="0" layer="19" extent="1-1"/>
 </signal>
-<signal name="N$18">
+<signal name="OUT6">
 <contactref element="OK1" pad="3"/>
 </signal>
-<signal name="N$22">
+<signal name="OUT7">
 <contactref element="OK1" pad="5"/>
 </signal>
-<signal name="N$27">
+<signal name="OUT8">
 <contactref element="OK1" pad="7"/>
 </signal>
@@
 <wire x1="-17.03100625" y1="-644.447175" x2="-6.876084375" y2="-221.22803125" width="0" layer="19" extent="1-1"/>
 </signal>
-<signal name="N$31">
+<signal name="OUT1">
 <contactref element="OK2" pad="1"/>
 </signal>
-<signal name="N$35">
+<signal name="OUT2">
 <contactref element="OK2" pad="3"/>
 </signal>
-<signal name="N$39">
+<signal name="OUT3">
 <contactref element="OK2" pad="5"/>
 </signal>
-<signal name="N$43">
+<signal name="OUT4">
 <contactref element="OK2" pad="7"/>
 </signal>
@@
 <contactref element="U$1" pad="HOLD"/>
 </signal>
+<signal name="L1-1">
+<contactref element="MOUT" pad="1"/>
+<contactref element="U$19" pad="1"/>
+<contactref element="U$20" pad="1"/>
+<contactref element="U$21" pad="1"/>
+<contactref element="U$22" pad="1"/>
+<wire x1="-15.811753125" y1="-655.32441875" x2="-20.84659375" y2="-670.0163125" width="0" layer="19" extent="1-1"/>
+<wire x1="-15.811753125" y1="-601.55564375" x2="-15.811753125" y2="-655.32441875" width="0" layer="19" extent="1-1"/>
+<wire x1="-15.811753125" y1="-547.786865625" x2="-15.811753125" y2="-601.55564375" width="0" layer="19" extent="1-1"/>
+<wire x1="-15.811753125" y1="-494.0180875" x2="-15.811753125" y2="-547.786865625" width="0" layer="19" extent="1-1"/>
+</signal>
+<signal name="MOUT1">
+<contactref element="MOUT" pad="2"/>
+<contactref element="U$19" pad="2"/>
+<wire x1="-19.621753125" y1="-494.0180875" x2="-15.84279375" y2="-670.0163125" width="0" layer="19" extent="1-1"/>
+</signal>
+<signal name="MOUT2">
+<contactref element="MOUT" pad="3"/>
+<contactref element="U$20" pad="2"/>
+<wire x1="-19.621753125" y1="-547.786865625" x2="-10.83899375" y2="-670.0163125" width="0" layer="19" extent="1-1"/>
+</signal>
+<signal name="MOUT3">
+<contactref element="MOUT" pad="4"/>
+<contactref element="U$21" pad="2"/>
+<wire x1="-19.621753125" y1="-601.55564375" x2="-5.83519375" y2="-670.0163125" width="0" layer="19" extent="1-1"/>
+</signal>
+<signal name="MOUT4">
+<contactref element="MOUT" pad="5"/>
+<contactref element="U$22" pad="2"/>
+<wire x1="-0.85679375" y1="-670.0163125" x2="-19.621753125" y2="-655.32441875" width="0" layer="19" extent="1-1"/>
+</signal>
+<signal name="L1-2">
+<contactref element="MOUT" pad="6"/>
+<contactref element="U$8" pad="1"/>
+<contactref element="U$16" pad="1"/>
+<contactref element="U$17" pad="1"/>
+<contactref element="U$18" pad="1"/>
+<wire x1="-15.811753125" y1="-366.66296875" x2="-15.811753125" y2="-420.431746875" width="0" layer="19" extent="1-1"/>
+<wire x1="-15.811753125" y1="-312.89419375" x2="-15.811753125" y2="-366.66296875" width="0" layer="19" extent="1-1"/>
+<wire x1="-15.811753125" y1="-67.225775" x2="-15.811753125" y2="-312.89419375" width="0" layer="19" extent="1-1"/>
+<wire x1="4.14700625" y1="-670.0163125" x2="-15.811753125" y2="-420.431746875" width="0" layer="19" extent="1-1"/>
+</signal>
+<signal name="MOUT5">
+<contactref element="MOUT" pad="7"/>
+<contactref element="U$8" pad="2"/>
+<wire x1="-19.621753125" y1="-67.225775" x2="9.15080625" y2="-670.0163125" width="0" layer="19" extent="1-1"/>
+</signal>
+<signal name="MOUT6">
+<contactref element="MOUT" pad="8"/>
+<contactref element="U$16" pad="2"/>
+<wire x1="-19.621753125" y1="-312.89419375" x2="14.15460625" y2="-670.0163125" width="0" layer="19" extent="1-1"/>
+</signal>
+<signal name="MOUT7">
+<contactref element="MOUT" pad="9"/>
+<contactref element="U$17" pad="2"/>
+<wire x1="-19.621753125" y1="-366.66296875" x2="19.15840625" y2="-670.0163125" width="0" layer="19" extent="1-1"/>
+</signal>
+<signal name="MOUT8">
+<contactref element="MOUT" pad="10"/>
+<contactref element="U$18" pad="2"/>
+<wire x1="24.16220625" y1="-670.0163125" x2="-19.621753125" y2="-420.431746875" width="0" layer="19" extent="1-1"/>
+</signal>
 </signals>

Commit message: Added microcontroller connections
Parts:
- added C1: 1000u, rcl:E5-8,5
- added C2: 0.1uF, rcl:C025-024X044
- added MIN, SV5: (no value), con-lstb:MA09-1
- added OLED_DISPLAY: (no value), con-lstb:MA04-1
- added PSU: (no value), con-ptr500:AK300/2
- added R1: 4.7K, rcl:0204/7
- added R2, R26: (no value), rcl:0204/7
- added R24, R25, R3, R4, R5, R6, R7: 330, rcl:0204/7
- added SV2: (no value), con-lstb:MA10-1
- added TEMP_SENSOR: (no value), con-lstb:MA03-1
- added X2: 22-23-2021, con-molex:22-23-2021
- added X3: Auto_Manual, con-molex:22-23-2021
- C5, C6, C7, C8: value (none) -> 0.1uF
- R10, R12, R14, R16, R18, R22, R8: value (none) -> 1k
- R11, R13, R15, R17, R19, R21, R23, R9: value (none) -> 150
- SV1: device con-lstb:MA09-1 -> con-lstb:MA10-1
- X1: value 22-23-2091 -> 22-23-2021; device con-molex:22-23-2091 -> con-molex:22-23-2021
- moved X1 130.9 mm to (-22.0, -833.3)
- moved SV1 115.4 mm to (-11.7, -802.9)
Connections:
- removed net CLK: U$1.CLK
- removed net DI: U$1.DI
- removed net DO: U$1.DO
- removed net N$23: U$1.HOLD
- removed net WP: U$1.WP
- new net AUTO: R2.2, SV2.10, X3.2
- new net FLASH_CLK: SV2.2, U$1.CLK
- new net FLASH_DI: SV2.3, U$1.DI
- new net FLASH_DO: SV2.4, U$1.DO
- new net IN1: R3.1, SV5.2
- new net IN2: R4.1, SV5.3
- new net IN3: R5.1, SV5.4
- new net IN4: R6.1, SV5.5
- new net IN5: R7.1, SV5.6
- new net IN6: R24.1, SV5.7
- new net IN7: R25.1, SV5.8
- new net IN8: R26.1, SV5.9
- new net N$1: SV1.1, X1.2
- new net N$14: SV1.10
- new net N$2: SV1.2, X2.2
- new net N$7: R24.2, R25.2, R26.2, R3.2, R4.2, R5.2, R6.2, R7.2
- new net N$8: SV5.1
- new net TEMP_SEN: R1.1, SV2.9, TEMP_SENSOR.2
- net +3V3: now also C2.1, OLED_DISPLAY.3, R1.2, TEMP_SENSOR.3, U$1.HOLD, U$1.WP, X2.1, X3.1
- net +5V: now also C1.+, PSU.1, X1.1
- net FLASH_CS: now also SV2.1
- net GND: now also C1.-, C2.2, MIN.1, OLED_DISPLAY.4, PSU.2, R2.1, SV1.3, SV1.4, SV1.5, SV1.6, TEMP_SENSOR.1
- net MISO: now also SV2.5
- net MOSI: now also SV2.6
- net OUT1: now also MIN.2
- net OUT2: now also MIN.3
- net OUT3: now also MIN.4
- net OUT4: now also MIN.5
- net OUT5: now also MIN.6
- net OUT6: now also MIN.7
- net OUT7: now also MIN.8
- net OUT8: now also MIN.9
- net SCK: now also SV2.7
- net SCL: now also OLED_DISPLAY.1
- net SDA: now also OLED_DISPLAY.2
- net SD_CS: now also SV2.8
- net SERIAL_RXD: now also SV1.7
- net SERIAL_TXD: now also SV1.8

Commit message: Finished first draft of the schematic, started organising the PCB
Parts:
- removed C5, C6, C7, C8: 0.1uF, rcl:C025-024X044
- removed LED1: (no value), led:LED3MM
- removed R10, R8: 1k, rcl:0204/7
- removed R11, R9: 150, rcl:0204/7
- removed S2: Reset, SparkFun:TACTILE_SWITCH_SMD
- removed U$16, U$8: SSR, HankLibraries:SSR_FOOTPRINT
- added 3.3V, 5V, LO5: (no value), led:LED3MM
- added CP02, CP14, CP22: 100n, rcl:E5-8,5
- added CP13, CP21: 100u, rcl:E5-8,5
- added C_BT, C_FM, C_RTC, C_USD: 0.1uF, rcl:C025-024X044
- added F1, F2, F3, F4, F5, F6, F7, F8: SM 092 A0 2A, fuse:PICOFUSE
- added LF33CV, LF50ABV: (no value), v-reg:78XXL
- added PR_3.3V, PR_5V, R62, RO52: 1k, rcl:0204/7
- added R51, R61: 150, rcl:0204/7
- added SSR5, SSR6: SSR, HankLibraries:SSR_FOOTPRINT
- CP01: value 1000u -> 100u
- moved MOUT 746.0 mm to (177.3, 55.0), turned to 90 degrees
- moved LED2 333.0 mm to (118.4, 7.86)
- moved OK1 298.2 mm to (95.0, 79.3), turned to 270 degrees
- moved OK2 260.2 mm to (94.5, 18.3), turned to 270 degrees
- moved U$1 108.5 mm to (41.3, 75.8)
- moved U$6 88.2 mm to (38.8, 26.8)
- moved U$7 81.0 mm to (42.6, -8.14)
- moved U$4 77.3 mm to (42.4, 47.8)
- moved SV5 66.1 mm to (-79.0, -1021.2)
- renumbered C1 to CP01, C2 to C_OLED, LED5 to LO1, LED6 to L_O2, LED7 to L_O3, LED8 to L_O4, R1 to R_TEMP, R12 to RO72, R13 to RO71, R14 to RO82, R15 to RO81, R16 to RO12, R17 to RO11, R18 to RO22, R19 to RO21, R20 to RO32, R21 to RO31, R22 to RO42, R23 to RO41, R24 to RI6, R25 to RI7, R26 to RI8, R3 to RI1, R4 to RI2, R5 to RI3, R6 to RI4, R7 to RI5, U$17 to SSR7, U$18 to SSR8, U$19 to SSR1, U$20 to SSR2, U$21 to SSR3, U$22 to SSR4
Connections:
- removed net MOUT1: MOUT.2, SSR1.2
- removed net N$34: L_O2.K, OK2.14, SSR2.4
- removed net N$38: L_O3.K, OK2.12, SSR3.4
- removed net RESET: S2.3, S2.4
- new net CP12: CP01.+, CP02.+, LF33CV.IN, LF50ABV.IN, PSU.1
- new net L_O1: L_O2.K, OK1.14, SSR2.4
- new net L_O3: L_O3.K, OK1.12, SSR3.4
- new net MO1: F1.2, MOUT.2
- new net MO2: F2.2, MOUT.3
- new net MO3: F3.2, MOUT.4
- new net MO4: F4.2, MOUT.5
- new net MO5: F5.2, MOUT.7
- new net MO6: F6.2, MOUT.8
- new net MO7: F7.2, MOUT.9
- new net MO8: F8.2, MOUT.10
- new net N$3: F1.1, SSR1.2
- new net N$4: 5V.K, PR_5V.2
- new net N$5: 3.3V.K, PR_3.3V.2
- net +3V3: now also 3.3V.A, CP21.+, CP22.+, C_BT.1, C_FM.1, C_RTC.2, C_USD.1, LF33CV.OUT; no longer C5.1, C6.1, C7.1, C8.2
- net +5V: now also 5V.A, CP13.+, CP14.+, LF50ABV.OUT, R62.2, RO52.2, SSR5.3, SSR6.3; no longer CP01.+, PSU.1, R10.2, R8.2, U$16.3, U$8.3
- net GND: now also CP02.-, CP13.-, CP14.-, CP21.-, CP22.-, C_BT.2, C_FM.2, C_RTC.1, C_USD.2, LF33CV.GND, LF50ABV.GND, PR_3.3V.1, PR_5V.1, R51.1, R61.1; no longer C5.2, C6.2, C7.2, C8.1, R11.1, R9.1, S2.1, S2.2
- net L1-2: now also SSR5.1, SSR6.1; no longer U$16.1, U$8.1
- net MOUT2: now also F2.1; no longer MOUT.3
- net MOUT3: now also F3.1; no longer MOUT.4
- net MOUT4: now also F4.1; no longer MOUT.5
- net MOUT5: now also F5.1, SSR5.2; no longer MOUT.7, U$8.2
- net MOUT6: now also F6.1, SSR6.2; no longer MOUT.8, U$16.2
- net MOUT7: now also F7.1; no longer MOUT.9
- net MOUT8: now also F8.1; no longer MOUT.10
- net N$11: now also LO5.A, RO52.1; no longer LED1.A, R8.1
- net N$12: now also LO5.K, OK2.16, SSR5.4; no longer LED1.K, OK1.16, U$8.4
- net N$15: now also OK2.2, R51.2; no longer OK1.2, R9.2
- net N$16: now also R62.1; no longer R10.1
- net N$17: now also OK2.14, SSR6.4; no longer OK1.14, U$16.4
- net N$19: now also OK2.4, R61.2; no longer OK1.4, R11.2
- net N$21: now also OK2.12; no longer OK1.12
- net N$24: now also OK2.6; no longer OK1.6
- net N$26: now also OK2.10; no longer OK1.10
- net N$28: now also OK2.8; no longer OK1.8
- net N$30: now also OK1.16; no longer OK2.16
- net N$32: now also OK1.2; no longer OK2.2
- net N$36: now also OK1.4; no longer OK2.4
- net N$40: now also OK1.6; no longer OK2.6
- net N$42: now also OK1.10; no longer OK2.10
- net N$44: now also OK1.8; no longer OK2.8
- net OUT1: now also OK1.1; no longer OK2.1
- net OUT2: now also OK1.3; no longer OK2.3
- net OUT3: now also OK1.5; no longer OK2.5
- net OUT4: now also OK1.7; no longer OK2.7
- net OUT5: now also OK2.1; no longer OK1.1
- net OUT6: now also OK2.3; no longer OK1.3
- net OUT7: now also OK2.5; no longer OK1.5
- net OUT8: now also OK2.7; no longer OK1.7
Routing:
- net RESET: track 39.0 -> 0.00 mm, vias 2 -> 0
- removed copper zone on layer 16, net GND
Other:
- board size 22.8 x 51.1 mm -> 7.6 x 134.9 mm

Commit message: Placed components in PCB and exported some pics to verify footprints
Parts:
- removed CP13, CP21: 100u, rcl:E5-8,5
- removed CP14, CP22: 100n, rcl:E5-8,5
- removed LED2, LED3, LED4: (no value), led:LED3MM
- removed SV5: (no value), con-lstb:MA09-1
- removed X1, X2: 22-23-2021, con-molex:22-23-2021
- added CP31, CP51: 100u, rcl:E5-8,5
- added CP32, CP52: 100n, rcl:E5-8,5
- added IN_BUTTONS: (no value), con-lstb:MA09-1
- added JUM_3.3V, JUM_5.5V: 22-23-2021, con-molex:22-23-2021
- added LO6, LO7, LO8: (no value), led:LED3MM
- moved PR_3.3V 1369.1 mm to (82.0, 36.6)
- moved 5V 1362.8 mm to (89.6, 28.2)
- moved 3.3V 1354.7 mm to (89.6, 37.4)
- moved PR_5V 1353.0 mm to (82.0, 27.4)
- moved LF33CV 1311.3 mm to (69.6, 29.3)
- moved LF50ABV 1311.0 mm to (53.1, 29.3)
- moved CP02 1299.8 mm to (34.0, 11.7)
- moved F8 1290.8 mm to (209.0, 47.1)
- moved F7 1285.8 mm to (209.0, 54.2)
- moved F6 1280.8 mm to (209.0, 61.3)
- moved F5 1277.1 mm to (209.0, 69.7)
- moved F4 1261.0 mm to (209.0, 77.6)
- moved F3 1256.0 mm to (209.0, 84.7)
- moved F2 1252.0 mm to (207.7, 93.1)
- moved F1 1128.9 mm to (209.0, 100.5)
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Connections:
- removed net N$8: SV5.1
- net +3V3: now also CP31.+, CP32.+, IN_BUTTONS.1, JUM_5.5V.1; no longer CP21.+, CP22.+, X2.1
- net +5V: now also CP51.+, CP52.+, JUM_3.3V.1; no longer CP13.+, CP14.+, X1.1
- net GND: now also CP31.-, CP32.-, CP51.-, CP52.-; no longer CP13.-, CP14.-, CP21.-, CP22.-
- net IN1: now also IN_BUTTONS.2; no longer SV5.2
- net IN2: now also IN_BUTTONS.3; no longer SV5.3
- net IN3: now also IN_BUTTONS.4; no longer SV5.4
- net IN4: now also IN_BUTTONS.5; no longer SV5.5
- net IN5: now also IN_BUTTONS.6; no longer SV5.6
- net IN6: now also IN_BUTTONS.7; no longer SV5.7
- net IN7: now also IN_BUTTONS.8; no longer SV5.8
- net IN8: now also IN_BUTTONS.9; no longer SV5.9
- net N$1: now also JUM_3.3V.2; no longer X1.2
- net N$16: now also LO6.A; no longer LED2.A
- net N$17: now also LO6.K; no longer LED2.K
- net N$2: now also JUM_5.5V.2; no longer X2.2
- net N$20: now also LO7.A; no longer LED3.A
- net N$21: now also LO7.K; no longer LED3.K
- net N$25: now also LO8.A; no longer LED4.A
- net N$26: now also LO8.K; no longer LED4.K
Other:
- board size 7.6 x 134.9 mm -> 256.5 x 110.8 mm

Commit message: Adding Arduino micro to the libraries, it will handle buttons and outputs. communication intended to be serial
Parts:
- moved F1 15.2 mm to (207.0, 115.6)
- moved SSR1 10.2 mm to (191.8, 110.5)
- moved U$7 9.45 mm to (69.8, 71.1)
- moved L_O4 5.64 mm to (156.2, 85.1)
- moved RO42 4.93 mm to (147.3, 85.1)
- moved RO32 4.50 mm to (147.3, 90.2)
- moved F2 4.36 mm to (212.1, 92.7)
- moved L_O3 3.95 mm to (156.2, 90.2)
- moved R_TEMP 3.81 mm to (68.1, 58.7)
- moved TEMP_SENSOR 3.81 mm to (67.0, 52.1)
- moved F7 3.10 mm to (212.1, 54.6)
- moved F3 3.10 mm to (212.1, 85.1)
- moved F6 3.09 mm to (212.1, 61.0)
- moved F5 3.08 mm to (212.1, 69.8)
- moved F4 3.07 mm to (212.1, 77.5)
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Other:
- board size 256.5 x 110.8 mm -> 256.5 x 129.5 mm

Commit message: Changed the interface of the SSR to Arduino. Added Arduino Sketch
Parts:
- removed MIN: (no value), con-lstb:MA09-1
- removed OK1, OK2: PC847, optocoupler:DIL16
- added ARDUINO: ARDUINO_MICRO, HankLibraries:ARDUINOMICRO_FOOTPRINT
- added RO13, RO23, RO43, RO53, RO73, RO83: 1k, rcl:0204/7
- added RO33: (no value), rcl:0204/7
- added RO62: 10K, rcl:0204/7
- added T1, T2, T3, T4, T5, T6, T7, T8: 2n2222, transistor:TO92-ECB
- R51, R61, RO11, RO71: value 150 -> 10K
- RO12, RO22, RO42, RO52, RO72, RO82: value 1k -> 10K
- RO32: value (none) -> 10K
- RO41, RO81: value 150 -> 10k
- moved RO32 334.3 mm to (-34.3, -190.5)
- moved RO22 331.3 mm to (-34.3, -203.2)
- moved RO42 319.5 mm to (-34.3, -177.8)
- moved RO72 283.9 mm to (-34.3, -152.4)
- moved RO52 271.3 mm to (-34.3, -127.0)
- moved RO82 270.4 mm to (-34.3, -165.1)
- moved RO12 220.9 mm to (-34.3, -25.4)
- renumbered R62 to RO63
Connections:
- removed net AUTO: R2.2, SV2.10, X3.2
- removed net N$32: OK1.2, RO11.2
- new net AUTO_MANUAL: ARDUINO.PB2, R2.2, SV2.10, X3.2
- new net N$18: RO62.1, T7.B
- new net N$22: RO72.1, T6.B
- new net N$23: RO42.1, T4.B
- new net N$27: RO32.1, T3.B
- new net N$31: RO22.1, T2.B
- new net N$34: RO82.1, T5.B
- new net N$35: ARDUINO.RX
- new net N$6: ARDUINO.TX
- new net N$8: RO12.1, T1.B
- new net N$9: RO52.1, T8.B
- net +5V: now also ARDUINO.VIN, RO13.2, RO23.2, RO33.2, RO43.2, RO53.2, RO73.2, RO83.2; no longer RO12.2, RO22.2, RO32.2, RO42.2, RO52.2, RO72.2, RO82.2
- net GND: now also ARDUINO.GND, ARDUINO.GND2, T3.E; no longer MIN.1, OK1.11, OK1.13, OK1.15, OK1.9, OK2.11, OK2.13, OK2.15, OK2.9
- net IN1: now also ARDUINO.PF7
- net IN2: now also ARDUINO.PF6
- net IN3: now also ARDUINO.PF5
- net IN4: now also ARDUINO.PF4
- net IN5: now also ARDUINO.PF1
- net IN6: now also ARDUINO.PF0
- net IN7: now also ARDUINO.PB3
- net IN8: now also ARDUINO.PB1
- net L_O1: now also T2.C; no longer OK1.14
- net L_O3: now also T3.C; no longer OK1.12
- net N$11: now also RO53.1; no longer RO52.1
- net N$12: now also T8.C; no longer OK2.16
- net N$15: now also RO52.2; no longer OK2.2
- net N$17: now also T7.C; no longer OK2.14
- net N$19: now also RO62.2; no longer OK2.4
- net N$20: now also RO73.1; no longer RO72.1
- net N$21: now also T6.C; no longer OK2.12
- net N$24: now also RO72.2; no longer OK2.6
- net N$25: now also RO83.1; no longer RO82.1
- net N$26: now also T5.C; no longer OK2.10
- net N$28: now also RO82.2; no longer OK2.8
- net N$29: now also RO13.1; no longer RO12.1
- net N$30: now also T1.C; no longer OK1.16
- net N$33: now also RO23.1; no longer RO22.1
- net N$36: now also RO22.2; no longer OK1.4
- net N$37: now also RO33.1; no longer RO32.1
- net N$40: now also RO32.2; no longer OK1.6
- net N$41: now also RO43.1; no longer RO42.1
- net N$42: now also T4.C; no longer OK1.10
- net N$44: now also RO42.2; no longer OK1.8
- net OUT1: now also ARDUINO.PC7, RO11.2, RO12.2; no longer MIN.2, OK1.1
- net OUT2: now also ARDUINO.PD6; no longer MIN.3, OK1.3
- net OUT3: now also ARDUINO.PB7; no longer MIN.4, OK1.5
- net OUT4: now also ARDUINO.PB6; no longer MIN.5, OK1.7
- net OUT5: now also ARDUINO.PB5; no longer MIN.6, OK2.1
- net OUT6: now also ARDUINO.PD7; no longer MIN.7, OK2.3
- net OUT7: now also ARDUINO.PC6; no longer MIN.8, OK2.5
- net OUT8: now also ARDUINO.PD0; no longer MIN.9, OK2.7

Commit message: Adding Arduino Serial communication and tiding up code
Parts:
- added TX1: 1k, rcl:0204/7
- added TX2: 2K, rcl:0204/7
- moved RO22 314.9 mm to (174.0, 33.0)
- moved RO32 314.9 mm to (174.0, 45.7)
- moved RO42 314.9 mm to (174.0, 58.4)
- moved RO52 314.9 mm to (174.0, 109.2)
- moved RO62 314.9 mm to (174.0, 96.5)
- moved RO72 314.9 mm to (174.0, 83.8)
- moved RO82 314.9 mm to (174.0, 71.1)
- moved T1 189.5 mm to (97.8, 121.9)
- moved T2 189.5 mm to (97.8, 96.5)
- moved T3 189.5 mm to (97.8, 83.8)
- moved T4 189.5 mm to (97.8, 71.1)
- moved T5 189.5 mm to (97.8, 58.4)
- moved T6 189.5 mm to (97.8, 45.7)
- moved T7 189.5 mm to (97.8, 33.0)
- moved T8 189.5 mm to (97.8, 20.3)
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Connections:
- net N$35 renamed ARD_RX
- new net ARD_TX: TX1.1, TX2.2
- net GND: now also TX2.1
- net N$6: now also TX1.2
