File: PCB/Hank2.sch (EAGLE design)
At the start: 114 parts, among them IC3 ATMEGA328-20P, T1 2n2222, T2 2n2222, T3 2n2222, T4 2n2222, T5 2n2222, T6 2n2222, T7 2n2222, T8 2n2222, X1 Sockets 1, X2 Sockets 2

Commit message: Updating parts footprint in the brd
Parts:
- removed CP02, CP32, CP52: 100n, rcl:CPOL-USE5-8.5
- added D_PSU: 1N4148DO35-7, diode:1N4148DO35-7
- CP31, CP51: value 100u -> 22uF
Connections:
- new net N$7: D_PSU.A, PSU-1.KL
- net +3V3: no longer CP32.+
- net +5V: no longer CP52.+
- net CP12: now also D_PSU.C; no longer CP02.+, PSU-1.KL
- net GND: no longer CP02.-, CP32.-, CP52.-
Other:
- moved on the sheet: CP01, CP31, CP51, PSU-1, PSU-2
Changed lines of the file:
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@@
 <part name="P+11" library="supply1" deviceset="+5V" device=""/>
 <part name="GND27" library="SparkFun" deviceset="GND" device=""/>
-<part name="CP52" library="rcl" deviceset="CPOL-US" device="E5-8.5" value="100n"/>
 <part name="+3V11" library="supply1" deviceset="+3V3" device=""/>
-<part name="CP02" library="rcl" deviceset="CPOL-US" device="E5-8.5" value="100n"/>
-<part name="CP51" library="rcl" deviceset="CPOL-US" device="E5-8.5" value="100u"/>
-<part name="CP31" library="rcl" deviceset="CPOL-US" device="E5-8.5" value="100u"/>
-<part name="CP32" library="rcl" deviceset="CPOL-US" device="E5-8.5" value="100n"/>
+<part name="CP51" library="rcl" deviceset="CPOL-US" device="E5-8.5" value="22uF"/>
+<part name="CP31" library="rcl" deviceset="CPOL-US" device="E5-8.5" value="22uF"/>
 <part name="D_3V3" library="led" deviceset="LED" device="3MM"/>
 <part name="PR_3.3V" library="rcl" deviceset="R-US_" device="0204/7" value="1k"/>
@@
 <part name="X1" library="con-ptr500" deviceset="AK300/5" device="" value="Sockets 1"/>
 <part name="X2" library="con-ptr500" deviceset="AK300/5" device="" value="Sockets 2"/>
+<part name="D_PSU" library="diode" deviceset="1N4148" device="DO35-7"/>
 </parts>
 <sheets>
@@
 <attribute name="VALUE" x="200.66" y="38.1" size="1.778" layer="96"/>
 </instance>
-<instance part="PSU" gate="-1" x="15.24" y="27.94"/>
-<instance part="PSU" gate="-2" x="15.24" y="10.16"/>
-<instance part="CP01" gate="G$1" x="22.86" y="20.32"/>
+<instance part="PSU" gate="-1" x="12.7" y="27.94"/>
+<instance part="PSU" gate="-2" x="12.7" y="10.16"/>
+<instance part="CP01" gate="G$1" x="33.02" y="17.78"/>
 <instance part="TEMP_SENSOR" gate="G$1" x="172.72" y="200.66" rot="MR0"/>
 <instance part="GND4" gate="1" x="142.24" y="195.58" smashed="yes">
@@
 <attribute name="VALUE" x="43.18" y="5.08" size="1.778" layer="96"/>
 </instance>
-<instance part="CP52" gate="G$1" x="68.58" y="20.32"/>
 <instance part="+3V11" gate="G$1" x="81.28" y="63.5"/>
-<instance part="CP02" gate="G$1" x="33.02" y="20.32"/>
-<instance part="CP51" gate="G$1" x="58.42" y="20.32"/>
-<instance part="CP31" gate="G$1" x="58.42" y="43.18"/>
-<instance part="CP32" gate="G$1" x="68.58" y="43.18"/>
+<instance part="CP51" gate="G$1" x="68.58" y="20.32"/>
+<instance part="CP31" gate="G$1" x="68.58" y="43.18"/>
 <instance part="D_3V3" gate="G$1" x="81.28" y="53.34"/>
 <instance part="PR_3.3V" gate="G$1" x="81.28" y="43.18" rot="R90"/>
@@
 <instance part="X2" gate="-4" x="370.84" y="139.7" rot="R180"/>
 <instance part="X2" gate="-5" x="370.84" y="160.02" rot="R180"/>
+<instance part="D_PSU" gate="G$1" x="20.32" y="27.94"/>
 </instances>
 <busses>
@@
 <wire x1="124.46" y1="254" x2="134.62" y2="254" width="0.1524" layer="91"/>
 <wire x1="134.62" y1="254" x2="139.7" y2="254" width="0.1524" layer="91"/>
-<wire x1="139.7" y1="254" x2="139.7" y2="248.92" width="0.1524" layer="91"/>
+<wire x1="139.7" y1="254" x2="129.54" y2="246.38" width="0.1524" layer="91"/>
 <pinref part="U$7" gate="G$1" pin="GND"/>
 <pinref part="C_USD" gate="G$1" pin="2"/>
@@
 <pinref part="PSU" gate="-2" pin="KL"/>
 <pinref part="CP01" gate="G$1" pin="-"/>
-<wire x1="20.32" y1="10.16" x2="22.86" y2="10.16" width="0.1524" layer="91"/>
-<wire x1="22.86" y1="10.16" x2="22.86" y2="15.24" width="0.1524" layer="91"/>
-<pinref part="CP02" gate="G$1" pin="-"/>
-<wire x1="33.02" y1="15.24" x2="33.02" y2="10.16" width="0.1524" layer="91"/>
-<wire x1="33.02" y1="10.16" x2="22.86" y2="10.16" width="0.1524" layer="91"/>
+<wire x1="17.78" y1="10.16" x2="33.02" y2="10.16" width="0.1524" layer="91"/>
+<wire x1="33.02" y1="10.16" x2="33.02" y2="12.7" width="0.1524" layer="91"/>
 <pinref part="GND27" gate="1" pin="GND"/>
 <wire x1="45.72" y1="20.32" x2="45.72" y2="10.16" width="0.1524" layer="91"/>
 <pinref part="CP51" gate="G$1" pin="-"/>
-<wire x1="58.42" y1="15.24" x2="58.42" y2="10.16" width="0.1524" layer="91"/>
-<wire x1="58.42" y1="10.16" x2="45.72" y2="10.16" width="0.1524" layer="91"/>
+<wire x1="68.58" y1="15.24" x2="68.58" y2="10.16" width="0.1524" layer="91"/>
+<wire x1="68.58" y1="10.16" x2="45.72" y2="10.16" width="0.1524" layer="91"/>
 <wire x1="33.02" y1="10.16" x2="45.72" y2="10.16" width="0.1524" layer="91"/>
 <pinref part="PR_5V" gate="G$1" pin="1"/>
 <wire x1="81.28" y1="10.16" x2="68.58" y2="10.16" width="0.1524" layer="91"/>
-<junction x="58.42" y="10.16"/>
-<pinref part="CP52" gate="G$1" pin="-"/>
-<wire x1="68.58" y1="10.16" x2="58.42" y2="10.16" width="0.1524" layer="91"/>
-<wire x1="68.58" y1="15.24" x2="68.58" y2="10.16" width="0.1524" layer="91"/>
 <junction x="68.58" y="10.16"/>
 <pinref part="REG_5V" gate="G$1" pin="GND"/>
 <junction x="33.02" y="10.16"/>
-<junction x="22.86" y="10.16"/>
 <junction x="45.72" y="10.16"/>
 </segment>
@@
 <pinref part="GND33" gate="1" pin="GND"/>
 <wire x1="68.58" y1="38.1" x2="81.28" y2="38.1" width="0.1524" layer="91"/>
-<pinref part="CP32" gate="G$1" pin="-"/>
 <pinref part="CP31" gate="G$1" pin="-"/>
-<wire x1="68.58" y1="38.1" x2="58.42" y2="38.1" width="0.1524" layer="91"/>
-<wire x1="58.42" y1="38.1" x2="45.72" y2="38.1" width="0.1524" layer="91"/>
-<junction x="58.42" y="38.1"/>
+<wire x1="68.58" y1="38.1" x2="45.72" y2="38.1" width="0.1524" layer="91"/>
 <junction x="68.58" y="38.1"/>
 <pinref part="REG_3V3" gate="G$1" pin="GND"/>
@@
 <net name="SCK" class="0">
 <segment>
-<wire x1="139.7" y1="228.6" x2="119.38" y2="228.6" width="0.1524" layer="91"/>
+<wire x1="129.54" y1="226.06" x2="119.38" y2="228.6" width="0.1524" layer="91"/>
 <pinref part="U$7" gate="G$1" pin="SCK"/>
 <label x="127" y="228.6" size="1.778" layer="95"/>
@@
 <net name="MISO" class="0">
 <segment>
-<wire x1="139.7" y1="238.76" x2="119.38" y2="238.76" width="0.1524" layer="91"/>
+<wire x1="129.54" y1="236.22" x2="119.38" y2="238.76" width="0.1524" layer="91"/>
 <pinref part="U$7" gate="G$1" pin="MISO"/>
 <label x="127" y="238.76" size="1.778" layer="95"/>
@@
 <net name="MOSI" class="0">
 <segment>
-<wire x1="139.7" y1="233.68" x2="119.38" y2="233.68" width="0.1524" layer="91"/>
+<wire x1="129.54" y1="231.14" x2="119.38" y2="233.68" width="0.1524" layer="91"/>
 <pinref part="U$7" gate="G$1" pin="MOSI"/>
 <label x="127" y="233.68" size="1.778" layer="95"/>
@@
 <net name="SD_CS" class="0">
 <segment>
-<wire x1="139.7" y1="223.52" x2="119.38" y2="223.52" width="0.1524" layer="91"/>
+<wire x1="129.54" y1="220.98" x2="119.38" y2="223.52" width="0.1524" layer="91"/>
 <pinref part="U$7" gate="G$1" pin="CS"/>
 <label x="127" y="223.52" size="1.778" layer="95"/>
@@
 </segment>
 <segment>
-<wire x1="139.7" y1="243.84" x2="134.62" y2="243.84" width="0.1524" layer="91"/>
+<wire x1="129.54" y1="241.3" x2="134.62" y2="243.84" width="0.1524" layer="91"/>
 <pinref part="+3V2" gate="G$1" pin="+3V3"/>
 <wire x1="134.62" y1="243.84" x2="119.38" y2="243.84" width="0.1524" layer="91"/>
@@
 <pinref part="+3V11" gate="G$1" pin="+3V3"/>
 <pinref part="D_3V3" gate="G$1" pin="A"/>
-<pinref part="CP32" gate="G$1" pin="+"/>
-<wire x1="58.42" y1="55.88" x2="68.58" y2="55.88" width="0.1524" layer="91"/>
 <wire x1="68.58" y1="55.88" x2="81.28" y2="55.88" width="0.1524" layer="91"/>
+<pinref part="CP31" gate="G$1" pin="+"/>
 <wire x1="68.58" y1="45.72" x2="68.58" y2="55.88" width="0.1524" layer="91"/>
-<pinref part="CP31" gate="G$1" pin="+"/>
-<wire x1="58.42" y1="45.72" x2="58.42" y2="55.88" width="0.1524" layer="91"/>
-<junction x="68.58" y="55.88"/>
 <junction x="81.28" y="55.88"/>
 <pinref part="REG_3V3" gate="G$1" pin="OUT"/>
-<wire x1="53.34" y1="55.88" x2="58.42" y2="55.88" width="0.1524" layer="91"/>
-<junction x="58.42" y="55.88"/>
+<wire x1="53.34" y1="55.88" x2="68.58" y2="55.88" width="0.1524" layer="91"/>
+<junction x="68.58" y="55.88"/>
 </segment>
 <segment>
@@
 </segment>
 <segment>
-<wire x1="53.34" y1="27.94" x2="58.42" y2="27.94" width="0.1524" layer="91"/>
-<pinref part="CP52" gate="G$1" pin="+"/>
-<wire x1="58.42" y1="27.94" x2="68.58" y2="27.94" width="0.1524" layer="91"/>
-<wire x1="68.58" y1="22.86" x2="68.58" y2="27.94" width="0.1524" layer="91"/>
+<wire x1="53.34" y1="27.94" x2="68.58" y2="27.94" width="0.1524" layer="91"/>
 <pinref part="P+11" gate="1" pin="+5V"/>
 <wire x1="81.28" y1="33.02" x2="81.28" y2="27.94" width="0.1524" layer="91"/>
 <pinref part="CP51" gate="G$1" pin="+"/>
 <wire x1="81.28" y1="27.94" x2="68.58" y2="27.94" width="0.1524" layer="91"/>
-<wire x1="58.42" y1="22.86" x2="58.42" y2="27.94" width="0.1524" layer="91"/>
+<wire x1="68.58" y1="22.86" x2="68.58" y2="27.94" width="0.1524" layer="91"/>
 <pinref part="D_5V" gate="G$1" pin="A"/>
 <junction x="81.28" y="27.94"/>
 <junction x="68.58" y="27.94"/>
-<junction x="58.42" y="27.94"/>
 <pinref part="REG_5V" gate="G$1" pin="OUT"/>
 </segment>
@@
 <net name="CP12" class="0">
 <segment>
-<pinref part="PSU" gate="-1" pin="KL"/>
 <pinref part="CP01" gate="G$1" pin="+"/>
-<wire x1="22.86" y1="22.86" x2="22.86" y2="27.94" width="0.1524" layer="91"/>
-<wire x1="22.86" y1="27.94" x2="20.32" y2="27.94" width="0.1524" layer="91"/>
+<wire x1="33.02" y1="20.32" x2="33.02" y2="27.94" width="0.1524" layer="91"/>
 <wire x1="38.1" y1="27.94" x2="33.02" y2="27.94" width="0.1524" layer="91"/>
-<pinref part="CP02" gate="G$1" pin="+"/>
-<wire x1="33.02" y1="27.94" x2="22.86" y2="27.94" width="0.1524" layer="91"/>
-<wire x1="33.02" y1="22.86" x2="33.02" y2="27.94" width="0.1524" layer="91"/>
 <wire x1="33.02" y1="27.94" x2="33.02" y2="55.88" width="0.1524" layer="91"/>
 <wire x1="33.02" y1="55.88" x2="38.1" y2="55.88" width="0.1524" layer="91"/>
 <pinref part="REG_5V" gate="G$1" pin="IN"/>
 <pinref part="REG_3V3" gate="G$1" pin="IN"/>
-<junction x="22.86" y="27.94"/>
 <junction x="33.02" y="27.94"/>
+<pinref part="D_PSU" gate="G$1" pin="C"/>
+<wire x1="22.86" y1="27.94" x2="33.02" y2="27.94" width="0.1524" layer="91"/>
 </segment>
 </net>
@@
 </segment>
 </net>
+<net name="N$7" class="0">
+<segment>
+<pinref part="D_PSU" gate="G$1" pin="A"/>
+<pinref part="PSU" gate="-1" pin="KL"/>
+</segment>
+</net>

Commit message: Changed the VRegs and Added a crowbar circuit to handle overvoltage conditions
Parts:
- removed URES: DTE6, switch-misc:DTE6
- added D_PSU1, D_PSU2: 1N4148DO35-7, diode:1N4148DO35-7
- added R1: (no value), rcl:R-US_0207/10
- added S1: DTS-6, switch-tact:DTS-6
- PR_3.3V, PR_5V, R51, R61, RDX, RI1, RI2, RI3, RI4, RI5, RI6, RI7, RI8, RO11, RO12, RO13, RO21, RO22, RO23, RO31, RO32, RO33, RO41, RO42, RO43, RO52, RO53, RO62, RO63, RO71, RO72, RO73, RO81, RO82, RO83, R_AUTO, R_NI1, R_NI2, R_TEMP, R_URES, R_UTX1, R_UTX2: device rcl:R-US_0204/7 -> rcl:R-US_0207/10
- REG_3V3: value LP2950CDT-3.3 -> AMS1117; device v-reg:LP2950CDT-3.3 -> AMS117:AMS1117
- REG_5V: value LP2950CDT-5.0 -> AMS1117; device v-reg:LP2950CDT-5.0 -> AMS117:AMS1117
Connections:
- net +3V3: now also D_PSU2.A, REG_3V3.OUT1
- net +5V: now also D_PSU1.A, REG_5V.OUT1
- net CP12: now also D_PSU1.C, D_PSU2.C
- net GND: now also S1.1, S1.2; no longer URES.P, URES.P@1
- net L1-1: now also SSR1.L2; no longer SSR1.L1
- net N$3: now also SSR1.L1; no longer SSR1.L2
- net U_RESET: now also S1.3, S1.4; no longer URES.S, URES.S@1
Other:
- moved on the sheet: CP31, CP51, D_5V, D_PSU, F1, F5, PR_5V, PSU-1, PSU-2

Commit message: Trying to set up the positions of the components in the PCB
Parts:
- removed R1: (no value), rcl:R-US_0207/10
- removed SV1, SV2: (no value), con-lstb:MA10-1
- added SV3: (no value), con-lstb:MA10-2
- PSU: device con-ptr500:AK300/2 -> con-ptr500:AK500/2
- X1, X2: device con-ptr500:AK300/5 -> con-ptr500:AK500/5
Connections:
- removed net MOUT2: F2.1, SSR2.L2
- removed net MOUT3: F3.1, SSR3.L2
- removed net MOUT4: F4.1, SSR4.L2
- removed net MOUT5: F5.1, SSR5.L2
- removed net MOUT6: F6.1, SSR6.L2
- removed net MOUT7: F7.1, SSR7.L2
- removed net MOUT8: F8.1, SSR8.L2
- new net N$10: F5.1, SSR5.L1
- new net N$13: F6.1, SSR6.L1
- new net N$14: F2.1, SSR2.L1
- new net N$15: F3.1, SSR3.L1
- new net N$19: F7.1, SSR7.L1
- new net N$24: F4.1, SSR4.L1
- new net N$28: F8.1, SSR8.L1
- net AUTO_MANUAL: now also SV3.20; no longer SV2.10
- net BT_RX: now also SV3.7; no longer SV1.4
- net BT_TX: now also SV3.9; no longer SV1.5
- net FLASH_CLK: now also SV3.4; no longer SV2.2
- net FLASH_CS: now also SV3.2; no longer SV2.1
- net FLASH_DI: now also SV3.6; no longer SV2.3
- net FLASH_DO: now also SV3.8; no longer SV2.4
- net GND: now also SV3.5; no longer SV1.3
- net L1-1: now also SSR2.L2, SSR3.L2, SSR4.L2; no longer SSR2.L1, SSR3.L1, SSR4.L1
- net L1-2: now also SSR5.L2, SSR6.L2, SSR7.L2, SSR8.L2; no longer SSR5.L1, SSR6.L1, SSR7.L1, SSR8.L1
- net MISO: now also SV3.10; no longer SV2.5
- net MOSI: now also SV3.12; no longer SV2.6
- net N$1: now also SV3.1; no longer SV1.1
- net N$2: now also SV3.3; no longer SV1.2
- net NEW_IN: now also SV3.11; no longer SV1.6
- net SCK: now also SV3.14; no longer SV2.7
- net SCL: now also SV3.19; no longer SV1.10
- net SDA: now also SV3.17; no longer SV1.9
- net SD_CS: now also SV3.16; no longer SV2.8
- net TEMP_SEN: now also SV3.18; no longer SV2.9
- net U_RX: now also SV3.13; no longer SV1.7
- net U_TX_3: now also SV3.15; no longer SV1.8
Other:
- moved on the sheet: F2, F3, F4, F5, F6, F7, F8
