File: PCB/Hank2.sch (EAGLE design)
At the start: 113 parts, among them IC3 ATMEGA328-20P, T1 2n2222, T2 2n2222, T3 2n2222, T4 2n2222, T5 2n2222, T6 2n2222, T7 2n2222, T8 2n2222, X1 Sockets 1, X2 Sockets 2

Commit message: PCB routing session
Connections:
- net +3V3: no longer AUTO-1.S, IN_BUTTONS.1
- net +5V: now also AUTO-1.S, IN_BUTTONS.9
- net IN1: now also IN_BUTTONS.1, RI1.1; no longer IN_BUTTONS.9, RI8.1
- net IN2: now also IN_BUTTONS.2, RI2.1; no longer IN_BUTTONS.8, RI7.1
- net IN3: now also IN_BUTTONS.3, RI3.1; no longer IN_BUTTONS.7, RI6.1
- net IN4: now also IN_BUTTONS.4, RI4.1; no longer IN_BUTTONS.6, RI5.1
- net IN5: now also RI5.1; no longer RI4.1
- net IN6: now also IN_BUTTONS.6, RI6.1; no longer IN_BUTTONS.4, RI3.1
- net IN7: now also IN_BUTTONS.7, RI7.1; no longer IN_BUTTONS.3, RI2.1
- net IN8: now also IN_BUTTONS.8, RI8.1; no longer IN_BUTTONS.2, RI1.1
- net L1-1: now also SSR1.L1, SSR2.L1, SSR3.L1, SSR4.L1; no longer SSR1.L2, SSR2.L2, SSR3.L2, SSR4.L2
- net L1-2: now also SSR5.L1, SSR6.L1, SSR7.L1, SSR8.L1; no longer SSR5.L2, SSR6.L2, SSR7.L2, SSR8.L2
- net MO1: now also X1-4.KL; no longer X1-1.KL
- net MO2: now also X1-3.KL; no longer X1-2.KL
- net MO3: now also X1-2.KL; no longer X1-3.KL
- net MO4: now also X1-1.KL; no longer X1-4.KL
- net MO5: now also X2-4.KL; no longer X2-1.KL
- net MO6: now also X2-3.KL; no longer X2-2.KL
- net MO7: now also X2-2.KL; no longer X2-3.KL
- net MO8: now also X2-1.KL; no longer X2-4.KL
- net N$10: now also F8.1, SSR8.L2; no longer F5.1, SSR5.L1
- net N$13: now also F7.1, SSR7.L2; no longer F6.1, SSR6.L1
- net N$14: now also SSR2.L2; no longer SSR2.L1
- net N$15: now also SSR3.L2; no longer SSR3.L1
- net N$19: now also F6.1, SSR6.L2; no longer F7.1, SSR7.L1
- net N$24: now also SSR4.L2; no longer SSR4.L1
- net N$28: now also F5.1, SSR5.L2; no longer F8.1, SSR8.L1
- net N$3: now also SSR1.L2; no longer SSR1.L1
Other:
- moved on the sheet: F1, F2, F3, F4, F5, F6, F7, F8, IN_BUTTONS, RI1, RI2, RI3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

Commit message: MAkng progress in the PCB
Parts:
- CP01, CP31, CP51: device rcl:CPOL-USE5-8.5 -> rcl:CPOL-EUE2.5-6
Connections:
- net N$6 renamed UTX
- net IN1: now also IN_BUTTONS.8; no longer IN_BUTTONS.1
- net IN2: now also IN_BUTTONS.7; no longer IN_BUTTONS.2
- net IN3: now also IN_BUTTONS.6; no longer IN_BUTTONS.3
- net IN4: now also IN_BUTTONS.5; no longer IN_BUTTONS.4
- net IN5: now also IN_BUTTONS.4; no longer IN_BUTTONS.5
- net IN6: now also IN_BUTTONS.3; no longer IN_BUTTONS.6
- net IN7: now also IN_BUTTONS.2; no longer IN_BUTTONS.7
- net IN8: now also IN_BUTTONS.1; no longer IN_BUTTONS.8
Other:
- moved on the sheet: RI1, RI2, RI3, RI4, RI5, RI6, RI7, RI8

Commit message: Finilised the pcb and sent to production
Parts:
- renumbered F1 to FUSE1, F2 to FUSE2, F3 to FUSE3, F4 to FUSE4, F5 to FUSE5, F6 to FUSE6, F7 to FUSE7, F8 to FUSE8, IC3 to IO_UC, J_3.3V to J_5V, J_5.5V to J_3V3V, L_O2 to LO2, L_O3 to LO3, L_O4 to LO4, S1 to U_RESET, SV3 to BREAKOUT, SV4 to JTAG, X1 to SKT1, X2 to SKT2
Other:
- note removed: "TO DO: +DONE Add connections to Microcontroller -Add 3.3V Power Supply Regulator -Add 5V low drop regulator +DONE: Add Temperature Sensor +DONE: Add the SSR Circuit -DONE:Add Fuses SM 092 A0 2A--- RS PN: 116-114 -Add Connector with 8Inputs http://www.gammon.com.au/images/Wire_Wrapped_Atmega132_e.png"
