File: PCB/Hank2.brd (EAGLE design)
At the start: 149.9 x 100.3 mm, 113 parts, among them IC3 ATMEGA328-20P, T1 2n2222, T2 2n2222, T3 2n2222, T4 2n2222, T5 2n2222, T6 2n2222, T7 2n2222, T8 2n2222, X1 Sockets 1, X2 Sockets 2

Commit message: PCB routing session
Parts:
- moved C_USD 121.9 mm to (91.4, 47.0)
- moved TEMP_SENSOR 111.9 mm to (53.3, 109.2)
- moved R_TEMP 106.6 mm to (48.3, 109.2)
- moved OLED_DISPLAY 81.8 mm to (50.8, 83.8)
- moved C_OLED 75.5 mm to (46.2, 79.5)
- moved R_NI1 74.2 mm to (35.6, 62.2), turned to 0 degrees
- moved U$4 69.9 mm to (24.1, 85.1), turned to 180 degrees
- moved R_NI2 68.3 mm to (35.6, 58.4), turned to 0 degrees
- moved RI1 67.9 mm to (86.4, 8.89), turned to 270 degrees
- moved R_AUTO 66.5 mm to (66.0, 8.89), turned to 90 degrees
- moved RI2 65.1 mm to (83.8, 8.89), turned to 270 degrees
- moved RI3 62.3 mm to (81.3, 8.89), turned to 270 degrees
- moved C_URTS 61.4 mm to (86.4, 36.8)
- moved RI4 59.7 mm to (78.7, 8.89), turned to 270 degrees
- moved RI5 57.2 mm to (76.2, 8.89), turned to 270 degrees
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Connections:
- net +3V3: no longer AUTO.1, IN_BUTTONS.1
- net +5V: now also AUTO.1, IN_BUTTONS.9
- net IN1: now also IN_BUTTONS.1, RI1.1; no longer IN_BUTTONS.9, RI8.1
- net IN2: now also IN_BUTTONS.2, RI2.1; no longer IN_BUTTONS.8, RI7.1
- net IN3: now also IN_BUTTONS.3, RI3.1; no longer IN_BUTTONS.7, RI6.1
- net IN4: now also IN_BUTTONS.4, RI4.1; no longer IN_BUTTONS.6, RI5.1
- net IN5: now also RI5.1; no longer RI4.1
- net IN6: now also IN_BUTTONS.6, RI6.1; no longer IN_BUTTONS.4, RI3.1
- net IN7: now also IN_BUTTONS.7, RI7.1; no longer IN_BUTTONS.3, RI2.1
- net IN8: now also IN_BUTTONS.8, RI8.1; no longer IN_BUTTONS.2, RI1.1
- net L1-1: now also SSR1.1, SSR2.1, SSR3.1, SSR4.1; no longer SSR1.2, SSR2.2, SSR3.2, SSR4.2
- net L1-2: now also SSR5.1, SSR6.1, SSR7.1, SSR8.1; no longer SSR5.2, SSR6.2, SSR7.2, SSR8.2
- net MO1: now also X1.4; no longer X1.1
- net MO2: now also X1.3; no longer X1.2
- net MO3: now also X1.2; no longer X1.3
- net MO4: now also X1.1; no longer X1.4
- net MO5: now also X2.4; no longer X2.1
- net MO6: now also X2.3; no longer X2.2
- net MO7: now also X2.2; no longer X2.3
- net MO8: now also X2.1; no longer X2.4
- net N$10: now also F8.1, SSR8.2; no longer F5.1, SSR5.1
- net N$13: now also F7.1, SSR7.2; no longer F6.1, SSR6.1
- net N$14: now also SSR2.2; no longer SSR2.1
- net N$15: now also SSR3.2; no longer SSR3.1
- net N$19: now also F6.1, SSR6.2; no longer F7.1, SSR7.1
- net N$24: now also SSR4.2; no longer SSR4.1
- net N$28: now also F5.1, SSR5.2; no longer F8.1, SSR8.1
- net N$3: now also SSR1.2; no longer SSR1.1
Other:
- board size 149.9 x 100.3 mm -> 168.9 x 119.4 mm

Commit message: MAkng progress in the PCB
Parts:
- CP01, CP31, CP51: device rcl:E5-8,5 -> rcl:E2,5-6
- moved C_USD 79.9 mm to (34.3, 102.9), turned to 270 degrees
- moved RO43 64.8 mm to (119.4, 5.08), turned to 180 degrees
- moved RO62 64.1 mm to (108.0, 99.1), turned to 180 degrees
- moved RO52 64.0 mm to (108.0, 111.8), turned to 180 degrees
- moved LO1 63.8 mm to (124.5, 52.1)
- moved RO13 62.2 mm to (119.4, 47.0), turned to 180 degrees
- moved RO33 62.2 mm to (119.4, 19.1), turned to 180 degrees
- moved RO23 62.2 mm to (119.4, 33.0), turned to 180 degrees
- moved RO11 62.0 mm to (108.0, 50.8), turned to 180 degrees
- moved RO12 62.0 mm to (108.0, 54.6), turned to 180 degrees
- moved RO22 61.8 mm to (108.0, 36.8), turned to 180 degrees
- moved T3 60.8 mm to (119.4, 24.1)
- moved T1 60.5 mm to (118.1, 52.1)
- moved T2 60.5 mm to (118.1, 38.1)
- moved RO21 60.5 mm to (108.0, 40.6), turned to 180 degrees
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Connections:
- net N$6 renamed UTX
- net IN1: now also IN_BUTTONS.8; no longer IN_BUTTONS.1
- net IN2: now also IN_BUTTONS.7; no longer IN_BUTTONS.2
- net IN3: now also IN_BUTTONS.6; no longer IN_BUTTONS.3
- net IN4: now also IN_BUTTONS.5; no longer IN_BUTTONS.4
- net IN5: now also IN_BUTTONS.4; no longer IN_BUTTONS.5
- net IN6: now also IN_BUTTONS.3; no longer IN_BUTTONS.6
- net IN7: now also IN_BUTTONS.2; no longer IN_BUTTONS.7
- net IN8: now also IN_BUTTONS.1; no longer IN_BUTTONS.8
Routing:
- net AUTO_MANUAL: track 0.00 -> 146.8 mm, vias 0 -> 1
- net OUT5: track 0.00 -> 125.5 mm
- net FLASH_CS: track 0.00 -> 117.6 mm
- net OUT6: track 0.00 -> 112.2 mm
- net FLASH_CLK: track 0.00 -> 112.1 mm
- net U_RX: track 0.00 -> 108.3 mm
- net FLASH_DI: track 0.00 -> 105.4 mm
- net OUT8: track 0.00 -> 98.2 mm
- net FLASH_DO: track 0.00 -> 97.1 mm
- net OUT7: track 0.00 -> 96.9 mm
- net NEW_IN: track 0.00 -> 94.0 mm
- net SCK: track 0.00 -> 84.2 mm
- net OUT4: track 0.00 -> 82.3 mm
- net U_RESET: track 0.00 -> 77.0 mm
- net TEMP_SEN: track 0.00 -> 74.6 mm
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- added copper zone on layer 16, net GND
- removed copper zone on layer 1, net GND

Commit message: Finilised the pcb and sent to production
Parts:
- removed F1, F2, F3, F4, F5, F6, F7, F8: SM 092 A0 2A, fuse:PICOFUSE
- removed X1: Sockets 1, con-ptr500:AK500/5
- removed X2: Sockets 2, con-ptr500:AK500/5
- added FUSE1, FUSE2, FUSE3, FUSE4, FUSE5, FUSE6, FUSE7, FUSE8: SM 092 A0 2A, fuse:PICOFUSE
- added SKT1: Sockets 1, con-ptr500:AK500/5
- added SKT2: Sockets 2, con-ptr500:AK500/5
- moved C_FM 10.8 mm to (95.9, 115.6)
- moved U$1 9.53 mm to (95.9, 108.0)
- moved R_TEMP 6.35 mm to (54.6, 101.6)
- moved TEMP_SENSOR 5.24 mm to (62.2, 104.1)
- moved XTALU 5.08 mm to (58.4, 48.3)
- moved C_UXTAL1 3.24 mm to (60.3, 54.0)
- moved C_UXTAL2 3.18 mm to (55.9, 54.0)
- moved T3 1.42 mm to (118.1, 24.8)
- moved IN_BUTTONS 1.27 mm to (72.4, 17.8)
- moved RI1 1.27 mm to (64.8, 8.89)
- moved RI2 1.27 mm to (67.3, 8.89)
- moved RI3 1.27 mm to (69.8, 8.89)
- moved RI4 1.27 mm to (72.4, 8.89)
- moved RI5 1.27 mm to (74.9, 8.89)
- moved RI6 1.27 mm to (77.5, 8.89)
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- renumbered IC3 to IO_UC, J_3.3V to J_5V, J_5.5V to J_3V3V, L_O2 to LO2, L_O3 to LO3, L_O4 to LO4, S1 to U_RESET, SV3 to BREAKOUT, SV4 to JTAG
Connections:
- net L1-1: now also SKT1.5; no longer X1.5
- net L1-2: now also SKT2.5; no longer X2.5
- net MO1: now also FUSE1.2, SKT1.4; no longer F1.2, X1.4
- net MO2: now also FUSE2.2, SKT1.3; no longer F2.2, X1.3
- net MO3: now also FUSE3.2, SKT1.2; no longer F3.2, X1.2
- net MO4: now also FUSE4.2, SKT1.1; no longer F4.2, X1.1
- net MO5: now also FUSE5.2, SKT2.4; no longer F5.2, X2.4
- net MO6: now also FUSE6.2, SKT2.3; no longer F6.2, X2.3
- net MO7: now also FUSE7.2, SKT2.2; no longer F7.2, X2.2
- net MO8: now also FUSE8.2, SKT2.1; no longer F8.2, X2.1
- net N$10: now also FUSE8.1; no longer F8.1
- net N$13: now also FUSE7.1; no longer F7.1
- net N$14: now also FUSE2.1; no longer F2.1
- net N$15: now also FUSE3.1; no longer F3.1
- net N$19: now also FUSE6.1; no longer F6.1
- net N$24: now also FUSE4.1; no longer F4.1
- net N$28: now also FUSE5.1; no longer F5.1
- net N$3: now also FUSE1.1; no longer F1.1
Routing:
- net +5V: track 0.00 -> 454.4 mm, vias 0 -> 1
- net +3V3: track 0.00 -> 257.5 mm, vias 0 -> 1
- net FLASH_DO: track 97.1 -> 135.7 mm
- net FLASH_CS: track 117.6 -> 154.7 mm
- net FLASH_DI: track 105.4 -> 141.9 mm
- net FLASH_CLK: track 112.1 -> 148.2 mm
- net GND: track 0.00 -> 34.1 mm
- net L1-1: track 53.1 -> 85.6 mm
- net SD_CS: track 57.3 -> 84.9 mm
- net OUT5: track 125.5 -> 147.9 mm
- net OUT6: track 112.2 -> 133.6 mm
- net OUT7: track 96.9 -> 115.4 mm
- net SCK: track 84.2 -> 100.3 mm
- net SCL: track 73.5 -> 58.5 mm, vias 0 -> 2
- net MOSI: track 70.3 -> 85.0 mm, vias 0 -> 3
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Other:
- board text added: "+5"
- board text added: "3V3"
- board text added: "5V"
- board text added: "ATMEGA328-20P"
- board text added: "AUTO/MANUAL"
- board text added: "Aut/Man"
- board text added: "BT_RX"
- board text added: "BT_TX"
- board text added: "DANGER"
- board text added: "DANGER LIVE MAINS"
- board text added: "FLASH_CLK"
- board text added: "FLASH_CS"
- board text added: "FLASH_DI"
- board text added: "FLASH_DO"
- board text added: "Freerangelobster.blogspot.co.uk https://github.com/FreeRangeLobster/FishHank Version 3.0 10/02/2020"
- board text added: "In1"
- board text added: "In2"
- board text added: "In3"
- board text added: "In4"
- board text added: "In5"
- board text added: "In6"
- board text added: "In7"
- board text added: "In8"
- board text added: "JLCJLCJLCJLC"
- board text added: "L1-1"
- board text added: "L1-2"
- board text added: "LINK"
- board text added: "LIVE MAINS"
- board text added: "MISO"
- board text added: "MOSI"
- board text added: "NEW_IN"
- board text added: "OUT1"
- board text added: "OUT2"
- board text added: "OUT3"
- board text added: "OUT4"
- board text added: "OUT5"
- board text added: "OUT6"
- board text added: "OUT7"
- board text added: "OUT8"
- board text added: "RESET"
- board text added: "RTS"
- board text added: "SCK"
- board text added: "SD_CS"
- board text added: "Temp_Sig"
- board text added: "URX"
- board text added: "UTX"
- board text added: "U_RX"
- board text added: "U_TX"
- board text added: "VIn"
- board text removed: "+5V"
- board text removed: "2012"
- board text removed: "DRDY"
- board text removed: "E:/Users/Ross/Desktop/Logo_nocolor.bmp"
- board text removed: "INT2"
- board text removed: "LSM303 Breakout^2"
- board text removed: "Ross Aiken"
- board text removed: "SA"
- board text removed: "Singularity"
- board text removed: "out"
